File: hardware/motor.kicad_sch (KiCad schematic)
At the start: 16 parts, among them J5 Conn_01x02_Socket, J6 Conn_01x02_Socket, J7 Conn_01x02_Socket, J8 Conn_01x02_Socket, Q1 AO3400A, Q2 AO3400A, Q3 AO3400A, Q4 AO3400A

Commit message: feat(kicad): Added several open sourced footprint libraries, finished schematic design for nrf, uwb, tof, flash, motors and added all reference material to refs folder
Other:
- note added: "Motor Driver"
Changed lines of the file:
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@@
+		)
+	)
+	(text "Motor Driver\n"
+		(exclude_from_sim no)
+		(at 194.31 89.154 0)
+		(effects
+			(font
+				(size 2.54 2.54)
+				(thickness 0.762)
+				(bold yes)
+			)
 		)
 	)
