File: hardware/uwb.kicad_sch (KiCad schematic)
At the start: 2 parts

Commit message: feat(kicad): Cleared ERC errors and assigned footprints for all parts
Parts:
- R21: footprint (none) -> Resistor_SMD:R_0402_1005Metric
Changed lines of the file:
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@@
-		)
-	)
-	(hierarchical_label "SPI2_MISO"
-		(shape output)
-		(at 26.67 29.21 180)
-		(effects
-			(font
-				(size 1.27 1.27)
-			)
-			(justify right)
 		)
 	)
@@
 			)
 			(justify left)
-		)
-	)
-	(hierarchical_label "SPI2_MOSI"
-		(shape input)
-		(at 26.67 26.67 180)
-		(effects
-			(font
-				(size 1.27 1.27)
-			)
-			(justify right)
-		)
-	)
-	(hierarchical_label "SPI2_SCK"
-		(shape input)
-		(at 26.67 21.59 180)
-		(effects
-			(font
-				(size 1.27 1.27)
-			)
-			(justify right)
 		)
 	)
@@
 			)
 		)
-		(property "Footprint" ""
+		(property "Footprint" "Resistor_SMD:R_0402_1005Metric"
 			(at 182.372 69.85 90)
 			(hide yes)

Commit message: feat(kicad): Added uwb application notes
Other:
- note added: "Application Notes 1)Chip Antenna should hang of the edge of the board 2) SPI traces should be as short as possible"
Changed lines of the file:
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@@
 	(rectangle
 		(start 88.9 49.53)
-		(end 205.74 127)
+		(end 205.74 137.16)
 		(stroke
 			(width 0.254)
@@
 		)
 	)
+	(text "Application Notes\n1)Chip Antenna should hang of the edge of the board\n2) SPI traces should be as short as possible"
+		(exclude_from_sim no)
+		(at 89.916 122.428 0)
+		(effects
+			(font
+				(size 1.27 1.27)
+			)
+			(justify left)
+		)
+	)
 	(text "Ultra Wide Band\n"
 		(exclude_from_sim no)
-		(at 188.976 124.968 0)
+		(at 189.23 134.62 0)
 		(effects
 			(font

Commit message: feat(kicad): Routing complete, assigning jlc components to each footprint
Parts:
- DWM1: now not fitted; now left out of the parts list
- R21: LCSC (none) -> C25741
Changed lines of the file:
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@@
 		(body_style 1)
 		(exclude_from_sim no)
-		(in_bom yes)
+		(in_bom no)
 		(on_board yes)
-		(in_pos_files yes)
-		(dnp no)
+		(in_pos_files no)
+		(dnp yes)
 		(fields_autoplaced yes)
 		(property "Reference" "DWM1"
@@
 		)
 		(property "Description" "Ultra wide band RF module With ranging location capabilities"
+			(at 146.05 86.36 0)
+			(hide yes)
+			(show_name no)
+			(do_not_autoplace no)
+			(effects
+				(font
+					(size 1.27 1.27)
+				)
+			)
+		)
+		(property "LCSC" ""
+			(at 146.05 86.36 0)
+			(hide yes)
+			(show_name no)
+			(do_not_autoplace no)
+			(effects
+				(font
+					(size 1.27 1.27)
+				)
+			)
+		)
+		(property "KLC_S3.3" ""
+			(at 146.05 86.36 0)
+			(hide yes)
+			(show_name no)
+			(do_not_autoplace no)
+			(effects
+				(font
+					(size 1.27 1.27)
+				)
+			)
+		)
+		(property "KLC_S4.1" ""
 			(at 146.05 86.36 0)
 			(hide yes)
@@
 			(at 184.15 69.85 0)
 			(hide yes)
+			(show_name no)
+			(do_not_autoplace no)
+			(effects
+				(font
+					(size 1.27 1.27)
+				)
+			)
+		)
+		(property "LCSC" "C25741"
+			(at 184.15 69.85 0)
+			(hide yes)
+			(show_name no)
+			(do_not_autoplace no)
+			(effects
+				(font
+					(size 1.27 1.27)
+				)
+			)
+		)
+		(property "KLC_S3.3" ""
+			(at 184.15 69.85 0)
+			(hide yes)
+			(show_name no)
+			(do_not_autoplace no)
+			(effects
+				(font
+					(size 1.27 1.27)
+				)
+			)
+		)
+		(property "KLC_S4.1" ""
+			(at 184.15 69.85 0)
+			(hide yes)
