File: hardware/radio.kicad_sch (KiCad schematic)
At the start: 17 parts, among them U7 nRF24L01P, Y1 16MHz (C13738)

Commit message: feat(kicad): Cleaned up routing and picked LCSC parts for several components
Parts:
- C28: footprint Capacitor_SMD:C_0402_1005Metric -> Capacitor_SMD:C_0603_1608Metric; LCSC (none) -> C21117
- C29: LCSC (none) -> C15195
- C30: LCSC (none) -> C1523
- C31: footprint Capacitor_SMD:C_0402_1005Metric -> Capacitor_SMD:C_0603_1608Metric; LCSC (none) -> C1604
- C32: LCSC (none) -> C1569
- C33: LCSC (none) -> C1552
- C34: LCSC (none) -> C1550
- C35, C36: LCSC (none) -> C1579
Changed lines of the file:
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@@
 			)
 		)
-		(property "Footprint" "Capacitor_SMD:C_0402_1005Metric"
+		(property "Footprint" "Capacitor_SMD:C_0603_1608Metric"
 			(at 182.5752 66.04 0)
 			(hide yes)
@@
 			)
 		)
-		(property "LCSC" ""
+		(property "LCSC" "C1604"
 			(at 181.61 62.23 0)
 			(hide yes)
@@
 			)
 		)
-		(property "LCSC" ""
+		(property "LCSC" "C1550"
 			(at 181.61 77.47 0)
 			(hide yes)
@@
 			)
 		)
-		(property "LCSC" ""
+		(property "LCSC" "C1523"
 			(at 121.92 48.26 0)
 			(hide yes)
@@
 			)
 		)
-		(property "LCSC" ""
+		(property "LCSC" "C1569"
 			(at 175.26 62.23 0)
 			(hide yes)
@@
 			)
 		)
-		(property "LCSC" ""
+		(property "LCSC" "C1552"
 			(at 171.45 73.66 90)
 			(hide yes)
@@
 			)
 		)
-		(property "LCSC" ""
+		(property "LCSC" "C1579"
 			(at 151.13 106.68 0)
 			(hide yes)
@@
 			)
 		)
-		(property "LCSC" ""
+		(property "LCSC" "C15195"
 			(at 115.57 48.26 0)
 			(hide yes)
@@
 			)
 		)
-		(property "LCSC" ""
+		(property "LCSC" "C1579"
 			(at 167.64 106.68 0)
 			(hide yes)
@@
 			)
 		)
-		(property "Footprint" "Capacitor_SMD:C_0402_1005Metric"
+		(property "Footprint" "Capacitor_SMD:C_0603_1608Metric"
 			(at 112.0648 102.87 0)
 			(hide yes)
@@
 			)
 		)
-		(property "LCSC" ""
+		(property "LCSC" "C21117"
 			(at 113.03 99.06 0)
 			(hide yes)
