File: hardware/swarm_drone.kicad_pcb (KiCad board)
At the start: 4 copper layers, 45 x 49 mm, 108 parts, among them J1 Conn_01x02_Pin, J2 Conn_01x03_Socket, J3 Conn_01x03_Socket, J5 Conn_01x02_Socket, J6 Conn_01x02_Socket, J7 Conn_01x02_Socket, J8 Conn_01x02_Socket, Q1 AO3400A, Q2 AO3400A, Q3 AO3400A, Q4 AO3400A, SW1 SW_Push, U1 STM32F405RGT7, U2 TPS7A91, U3 ICM-42688-P, U4 BMP581, U5 VL53L1CXV0FY1, U6 GD25Q128ESIGR, U7 nRF24L01P, X1 8MHz, Y1 16MHz (C13738)

Commit message: feat(kicad): Routing complete, assigning jlc components to each footprint
Parts:
- removed the C20 at (111.9, 52.6)
- removed the C20 at (110.3, 52.2)
- removed J2, J3: Conn_01x03_Socket, Connector_PinHeader_1.00mm:PinHeader_1x03_P1.00mm_Horizontal
- added C20: 100n, Capacitor_SMD:C_0402_1005Metric, F.Cu at (112.0, 52.6)
- added C38: 100n, Capacitor_SMD:C_0402_1005Metric, F.Cu at (92.6, 64.3)
- added J4: SM03B-SRSS-TB_LF__SN_ (C160403), header:JST_SM03B-SRSS-TB_LF__SN_, F.Cu at (117.9, 56.2)
- added J9: SM03B-SRSS-TB_LF__SN_ (C160403), header:JST_SM03B-SRSS-TB_LF__SN_, F.Cu at (117.9, 49.8)
- C17: value 0.1u -> 100n
- C18: value 2.2u -> 2u2
- C22, C23: value 26p -> 27p
- C8, C9: value 1u -> 2u2
- R12, R13, R14, R15: value 10k -> 4k7
- R22, R23, R24, R25, R26, R27: value 330R -> 2k2
- R3: value 3.57k -> 4k7
- R4: value 1.15k -> 1k5
- moved R13 0.95 mm to (116.6, 49.4)
- moved Q2 0.91 mm to (119.4, 49.1)
- moved Q3 0.87 mm to (119.9, 74.8)
- moved D3 0.60 mm to (114.8, 80.6)
- moved D1 0.49 mm to (87.0, 43.7)
- moved R23 0.48 mm to (111.2, 59.8)
- moved R15 0.43 mm to (87.4, 74.7)
- moved R27 0.42 mm to (111.2, 65.2)
- moved R26 0.37 mm to (111.1, 63.9)
- moved J7 0.35 mm to (119.9, 81.0)
- moved D8 0.34 mm to (113.7, 62.4)
- moved D5 0.34 mm to (113.8, 56.8)
- moved D7 0.33 mm to (113.8, 60.7)
- moved D6 0.33 mm to (113.8, 58.9)
- moved D9 0.32 mm to (113.8, 64.2)
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Connections:
- L1 pad 2: GND -> /Radio/VDD_PA
- R17 pad 2: Net-(U5-XSHUT) -> /Microcontroller/VL53L1X_XSHUT
- U1 pad 17: /IMU/IMU_CS -> /IMU/IMU_INT
- U1 pad 20: /IMU/IMU_INT -> /IMU/IMU_CS
- U1 pad 9: unconnected-(U1-PC1-Pad9) -> /Microcontroller/VL53L1X_XSHUT
- U5 pad 5: Net-(U5-XSHUT) -> /Microcontroller/VL53L1X_XSHUT
Routing:
- net /Microcontroller/VL53L1X_XSHUT: track 0.00 -> 13.2 mm, vias 0 -> 1
- net /IMU/IMU_CS: track 11.0 -> 17.5 mm
- net /IMU/IMU_INT: track 9.12 -> 3.84 mm
- net /Microcontroller/USART1_TX: track 17.1 -> 12.0 mm
- net /Microcontroller/SWCLK: track 20.2 -> 15.5 mm
- net /Microcontroller/USART1_RX: track 16.4 -> 13.3 mm
- net /Microcontroller/M2: track 23.8 -> 22.1 mm
- net +3V3: track 81.9 -> 80.2 mm
- net Net-(U5-XSHUT): track 1.51 -> 0.00 mm
- net Net-(D3-A): track 8.55 -> 10.0 mm
- net Net-(D4-A): track 9.66 -> 8.35 mm
- net /Microcontroller/SWDIO: track 17.1 -> 15.8 mm
- net Net-(D2-A): track 9.05 -> 8.32 mm
- net /Microcontroller/M3: track 21.4 -> 20.7 mm
- net GND: track 160.4 -> 161.0 mm, vias 46 -> 76
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Other:
- board text added: "G"
- board text removed: "Memory"
- board text removed: "SWCLK"

Commit message: feat(kicad): Cleaned up routing and picked LCSC parts for several components
Parts:
- C28, C31: footprint Capacitor_SMD:C_0402_1005Metric -> Capacitor_SMD:C_0603_1608Metric
- moved C28 0.68 mm to (97.4, 48.7)
- moved C21 0.62 mm to (113.1, 53.9)
- moved C20 0.60 mm to (111.4, 52.5)
- moved C22 0.50 mm to (91.7, 51.3)
- moved C31 0.47 mm to (104.1, 41.9)
- moved SW1 0.12 mm to (87.1, 56.5)
- moved R2 0.08 mm to (86.5, 52.9)
- moved C10 0.07 mm to (86.5, 51.9)
- moved R27 0.06 mm to (111.2, 65.1)
Routing:
- net GND: track 161.0 -> 168.0 mm, vias 76 -> 85
- net /Barometer/SPI3_MISO: track 21.9 -> 21.1 mm
- net /Barometer/SPI3_MOSI: track 21.8 -> 21.1 mm
- net +BATT: track 180.9 -> 181.7 mm
Other:
- board text added: "ALT RADIO"
- board text added: "RST"
- board text removed: "RADIO EXT"
